File: Assets/PCB Files/UGV.kicad_pcb (KiCad board)
At the start: 2 copper layers, 120.6 x 156.5 mm, 78 parts, among them J13 USB3_A, J15 Screw_Terminal_01x12, J16 Screw_Terminal_01x12, J17 Screw_Terminal_01x12, J18 Screw_Terminal_01x12, Q1 AO3400A, U2 LMR33630ADDA, U3 SN74LVC8T245, U4 Teensy4.1, U5 SN74LVC8T245

Commit message: Updated
Routing:
- net /Vout: track 206.6 -> 239.5 mm
- net Net-(12Vout1-PadP): track 39.0 -> 55.2 mm
