File: Assets/PCB Files/.history/UGV.kicad_sch (KiCad schematic)
At the start: 95 parts, among them J13 USB3_A, J15 Screw_Terminal_01x12, J16 Screw_Terminal_01x12, J17 Screw_Terminal_01x12, J18 Screw_Terminal_01x12, Q1 AO3400A, Q2 AO3400A, Q3 AO3400A, U2 LMR33630ADDA, U3 SN74LVC8T245, U4 Teensy4.1, U5 SN74LVC8T245

Commit message: Routing changes in the LMR IC and a few small changes too
Parts:
- 12Vout(C)1, 12Vout1, BUCKin1, BUCKout1, Contactor1, EByte1, Jetson1, PWRout1, Ubiquiti1: MPN XT30PW-M -> (none)
- 5Vout1, 5Vout2, EncPWR1, EncPWR2, EncPWR3, EncPWR4, LED1, Laser1, Relay1, Servo1, Servo2: MPN B2B-XH-A -> (none)
- C12, C7, Cout1, Cout2: MPN C1210C226K3RACTU -> (none)
- Enc1, Enc2, Enc3, Enc4: MPN B2B-XH-A-BK -> (none)
- Fan1, Fan2, Fan3, Fan4: MPN B2B-XH-A-R -> (none)
- Flysky1, Flysky2, MDDS30_DIR1, MDDS30_PWM1, MDDS30_PWM2: MPN B4B-XH-A (LF)(SN) -> (none)
- PWRin1: footprint Connector_AMASS:AMASS_XT90PW-M_1x02_P10.90mm_Horizontal -> UGV_Custom:AMASS_XT90PW-M_1x02_P10.90mm_Horizontal
- U2: MPN (none) -> LMR33630ADDAR
Changed lines of the file:
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@@
 			)
 		)
-		(property "MPN" "B2B-XH-A"
+		(property "MPN" ""
 			(at 24.13 176.53 90)
 			(hide yes)
@@
 			)
 		)
-		(property "MPN" "XT30PW-M"
+		(property "MPN" ""
 			(at 29.21 97.79 0)
 			(hide yes)
@@
 			)
 		)
-		(property "MPN" "B2B-XH-A"
+		(property "MPN" ""
 			(at 81.28 176.53 90)
 			(hide yes)
@@
 			)
 		)
-		(property "MPN" "B2B-XH-A-BK"
+		(property "MPN" ""
 			(at 254 135.89 0)
 			(hide yes)
@@
 			)
 		)
-		(property "MPN" "B2B-XH-A"
+		(property "MPN" ""
 			(at 154.94 177.8 90)
 			(hide yes)
@@
 			)
 		)
-		(property "MPN" "XT30PW-M"
+		(property "MPN" ""
 			(at 29.21 24.13 0)
 			(hide yes)
@@
 			)
 		)
-		(property "MPN" "B2B-XH-A-BK"
+		(property "MPN" ""
 			(at 254 115.57 0)
 			(hide yes)
@@
 			)
 		)
-		(property "MPN" "B4B-XH-A (LF)(SN)"
+		(property "MPN" ""
 			(at 275.59 45.72 0)
 			(hide yes)
@@
 			)
 		)
-		(property "MPN" "C1210C226K3RACTU"
+		(property "MPN" ""
 			(at 128.27 133.35 0)
 			(hide yes)
@@
 			)
 		)
-		(property "MPN" "XT30PW-M"
+		(property "MPN" ""
 			(at 29.21 154.94 0)
 			(hide yes)
@@
 			)
 		)
-		(property "MPN" "XT30PW-M"
+		(property "MPN" ""
 			(at 29.21 64.77 0)
 			(hide yes)
@@
 			)
 		)
-		(property "MPN" "C1210C226K3RACTU"
+		(property "MPN" ""
 			(at 120.65 133.35 0)
 			(hide yes)
@@
 			)
 		)
-		(property "MPN" "C1210C226K3RACTU"
+		(property "MPN" ""
 			(at 86.36 27.94 0)
 			(hide yes)
@@
 			)
 		)
-		(property "MPN" "B2B-XH-A"
+		(property "MPN" ""
 			(at 171.5397 168.9036 90)
 			(hide yes)
@@
 			)
 		)
-		(property "MPN" "C1210C226K3RACTU"
+		(property "MPN" ""
 			(at 54.61 27.94 0)
 			(hide yes)
@@
 			)
 		)
-		(property "MPN" "B4B-XH-A (LF)(SN)"
+		(property "MPN" ""
 			(at 275.59 66.04 0)
 			(hide yes)
@@
 			)
 		)
-		(property "MPN" "B4B-XH-A (LF)(SN)"
+		(property "MPN" ""
 			(at 220.98 17.78 0)
 			(hide yes)
@@
 			)
 		)
-		(property "MPN" "B2B-XH-A"
+		(property "MPN" ""
 			(at 67.31 176.53 90)
 			(hide yes)
@@
 			)
 		)
-		(property "MPN" "XT30PW-M"
+		(property "MPN" ""
 			(at 135.89 16.51 0)
 			(hide yes)
@@
 			)
 		)
-		(property "MPN" "B2B-XH-A-R"
+		(property "MPN" ""
 			(at 34.29 130.81 90)
 			(hide yes)
@@
 			)
 		)
-		(property "Footprint" "Connector_AMASS:AMASS_XT90PW-M_1x02_P10.90mm_Horizontal"
+		(property "Footprint" "UGV_Custom:AMASS_XT90PW-M_1x02_P10.90mm_Horizontal"
 			(at 29.21 74.93 0)
 			(hide yes)
@@
 			)
 		)
-		(property "MPN" "B4B-XH-A (LF)(SN)"
+		(property "MPN" ""
 			(at 190.5 17.78 0)
 			(hide yes)
@@
 			)
 		)
-		(property "MPN" "B2B-XH-A"
+		(property "MPN" ""
 			(at 52.07 176.53 90)
 			(hide yes)
@@
 			)
 		)
+		(property "MPN" "LMR33630ADDAR"
+			(at 74.93 134.62 0)
+			(hide yes)
+			(show_name no)
+			(do_not_autoplace no)
+			(effects
+				(font
+					(size 1.27 1.27)
+				)
+			)
+		)
 		(pin "3"
 		)
@@
 			)
 		)
-		(property "MPN" "XT30PW-M"
+		(property "MPN" ""
 			(at 124.46 16.51 0)
 			(hide yes)
@@
 			)
 		)
-		(property "MPN" "B2B-XH-A"
+		(property "MPN" ""
 			(at 213.36 168.91 90)
 			(hide yes)
@@
 			)
 		)
-		(property "MPN" "XT30PW-M"
+		(property "MPN" ""
 			(at 29.21 36.83 0)
 			(hide yes)
@@
 			)
 		)
-		(property "MPN" "B2B-XH-A-R"
+		(property "MPN" ""
 			(at 34.29 140.97 90)
 			(hide yes)
@@
 			)
 		)
-		(property "MPN" "XT30PW-M"
+		(property "MPN" ""
 			(at 29.21 86.36 0)
 			(hide yes)
@@
 			)
 		)
-		(property "MPN" "B2B-XH-A-R"
+		(property "MPN" ""
 			(at 34.29 120.65 90)
 			(hide yes)
@@
 			)
 		)
-		(property "MPN" "B2B-XH-A"
+		(property "MPN" ""
 			(at 38.1 176.53 90)
 			(hide yes)
@@
 			)
 		)
-		(property "MPN" "B2B-XH-A-BK"
+		(property "MPN" ""
 			(at 254 125.73 0)
 			(hide yes)
@@
 			)
 		)
-		(property "MPN" "B2B-XH-A-R"
+		(property "MPN" ""
 			(at 34.29 110.49 90)
 			(hide yes)
@@
 			)
 		)
-		(property "MPN" "XT30PW-M"
+		(property "MPN" ""
 			(at 29.21 49.53 0)
 			(hide yes)
@@
 			)
 		)
-		(property "MPN" "B2B-XH-A"
+		(property "MPN" ""
 			(at 199.39 168.91 90)
 			(hide yes)
@@
 			)
 		)
-		(property "MPN" "B2B-XH-A-BK"
+		(property "MPN" ""
 			(at 254 146.05 0)
 			(hide yes)
@@
 			)
 		)
-		(property "MPN" "B4B-XH-A (LF)(SN)"
+		(property "MPN" ""
 			(at 175.26 17.78 0)
 			(hide yes)
@@
 			)
 		)
-		(property "MPN" "B2B-XH-A"
+		(property "MPN" ""
 			(at 185.42 168.7568 90)
 			(hide yes)
@@
 			)
 		)
-		(property "MPN" "B2B-XH-A"
+		(property "MPN" ""
 			(at 95.25 176.53 90)
 			(hide yes)
